Commit message: Fixing up cde

File: description/robot_core.xacro (robot description, xacro)
@@ -1,31 +1,31 @@
 <?xml version="1.0"?>
 <robot xmlns:xacro="http://www.ros.org/wiki/xacro" >
-    <material name="white">
-    color rgba="1 1 1 1"
+    xacro <material name="white">
+        xacro <color rgba="1.0 1.0 1.0 1.0"/>
     </material>
-    <material name="orange">
-    color rgba="1 0.3 0.1 1"
+    xacro <material name="orange">
+        xacro <color rgba="1 0.3 0.1 1"/>
     </material>
-    <material name="blue">
-    color rgba="0.2 0.2 1 1"
+    xacro <material name="blue">
+        xacro <color rgba="0.2 0.2 1 1"/>
     </material>
-    <material name="black">
-    color rgba="0 0 0 1"
+    xacro <material name="black">
+        xacro <color rgba="0 0 0 1"/>
     </material>
     <link name="base_link">
     </link>
     <joint name="chassis_joint" type="fixed">
-    <parent link="base_link"/>
-    <child link="chassis"/>
-    <origin xyz="-0.1 0 0"/>
+        <parent link="base_link"/>
+        <child link="chassis"/>
+        <origin xyz="-0.1 0 0"/>
     </joint>
     <link name="chassis">
-    <visual>
-    <geometry>
-    <origin xyz="0.15 0 0.075"/>
-    <box size ="0.3 0.3 0.15"/>
-    </geometry>
-    <material name="white"/>
-    </visual>
+        <visual>
+            xacro:<origin xyz="0.15 0 0.075"/>
+            xacro <geometry>
+                xacro <box size ="0.3 0.3 0.15"/>
+            </geometry>
+            <material name="white"/>
+        </visual>
     </link>
 </robot>

Commit message: fixing up code

File: description/robot_core.xacro (robot description, xacro)
@@ -22,5 +22,5 @@
     <link name="chassis">
         <visual>
-            xacro:<origin xyz="0.15 0 0.075"/>
+            xacro <origin xyz="0.15 0 0.075"/>
             xacro <geometry>
                 xacro <box size ="0.3 0.3 0.15"/>

Commit message: Aadding wheels

File: description/robot_core.xacro (robot description, xacro)
@@ -13,6 +13,8 @@
         xacro <color rgba="0 0 0 1"/>
     </material>
+    <!-- BASE LINK -->
     <link name="base_link">
     </link>
+   <!-- CHASSIS  -->
     <joint name="chassis_joint" type="fixed">
         <parent link="base_link"/>
@@ -29,3 +31,35 @@
         </visual>
     </link>
+       <!-- left wheel link  -->
+    <joint name="left_wheel_joint" type="continous">
+        <parent link="base_link"/>
+        <child link="left_wheel"/>
+        <origin xyz="0 0.175 0" rpy="-${pi/2} 0 0"/>
+        <axis xyz="0 0 1"/>
+    </joint>
+    <link name="left_wheel">
+        <visual>
+            xacro <origin xyz="0.15 0 0.075"/>
+            xacro <geometry>
+                xacro <cylinder radius="0.05" length="0.04"/>
+            </geometry>
+            <material name="blue"/>
+        </visual>
+    </link>
+           <!-- RIGHT WHEEL LINK  -->
+    <joint name="right_wheel_joint" type="continous">
+        <parent link="base_link"/>
+        <child link="right_wheel"/>
+        <origin xyz="0 0.175 0" rpy="${pi/2} 0 0"/>
+        <axis xyz="0 0 -1"/>
+    </joint>
+    <link name="right_wheel">
+         <visual>
+            xacro <origin xyz="0.15 0 0.075"/>
+             xacro <geometry>
+                  xacro <cylinder radius="0.05" length="0.04"/>
+            </geometry>
+            <material name="blue"/>
+        </visual>
+    </link>
 </robot>

Commit message: adding more wheels

File: description/robot_core.xacro (robot description, xacro)
@@ -32,5 +32,5 @@
     </link>
        <!-- left wheel link  -->
-    <joint name="left_wheel_joint" type="continous">
+    <joint name="left_wheel_joint" type="continuous">
         <parent link="base_link"/>
         <child link="left_wheel"/>
@@ -48,8 +48,8 @@
     </link>
            <!-- RIGHT WHEEL LINK  -->
-    <joint name="right_wheel_joint" type="continous">
+    <joint name="right_wheel_joint" type="continuous">
         <parent link="base_link"/>
         <child link="right_wheel"/>
-        <origin xyz="0 0.175 0" rpy="${pi/2} 0 0"/>
+        <origin xyz="0 -0.175 0" rpy="${pi/2} 0 0"/>
         <axis xyz="0 0 -1"/>
     </joint>

Commit message: adding wheels without xacro

File: description/robot_core.xacro (robot description, xacro)
@@ -31,35 +31,32 @@
         </visual>
     </link>
-       <!-- left wheel link  -->
-    <joint name="left_wheel_joint" type="continuous">
-        <parent link="base_link"/>
-        <child link="left_wheel"/>
-        <origin xyz="0 0.175 0" rpy="-${pi/2} 0 0"/>
-        <axis xyz="0 0 1"/>
-    </joint>
-    <link name="left_wheel">
-        <visual>
-            xacro <origin xyz="0.15 0 0.075"/>
-            xacro <geometry>
-                xacro <cylinder radius="0.05" length="0.04"/>
-            </geometry>
-            <material name="blue"/>
-        </visual>
-    </link>
-           <!-- RIGHT WHEEL LINK  -->
-    <joint name="right_wheel_joint" type="continuous">
-        <parent link="base_link"/>
-        <child link="right_wheel"/>
-        <origin xyz="0 -0.175 0" rpy="${pi/2} 0 0"/>
-        <axis xyz="0 0 -1"/>
-    </joint>
-    <link name="right_wheel">
-         <visual>
-            xacro <origin xyz="0.15 0 0.075"/>
-             xacro <geometry>
-                  xacro <cylinder radius="0.05" length="0.04"/>
-            </geometry>
-            <material name="blue"/>
-        </visual>
-    </link>
+      <!-- LEFT WHEEL -->
+<joint name="left_wheel_joint" type="continuous">
+    <parent link="base_link"/>
+    <child link="left_wheel"/>
+    <origin xyz="0 0.175 0" rpy="-${pi/2} 0 0"/>
+    <axis xyz="0 0 1"/>
+</joint>
+<link name="left_wheel">
+    <visual>
+        <geometry>
+            <cylinder length="0.04" radius="0.05" />
+        </geometry>
+        <material name="blue"/>
+    </visual>
+</link>
+<joint name="right_wheel_joint" type="continuous">
+    <parent link="base_link"/>
+    <child link="right_wheel"/>
+    <origin xyz="0 -0.175 0" rpy="${pi/2} 0 0"/>
+    <axis xyz="0 0 -1"/>
+</joint>
+<link name="right_wheel">
+    <visual>
+        <geometry>
+            <cylinder length="0.04" radius="0.05" />
+        </geometry>
+        <material name="blue"/>
+    </visual>
+</link>
 </robot>

Commit message: Adding the casto wheel

File: description/robot_core.xacro (robot description, xacro)
@@ -46,4 +46,5 @@
     </visual>
 </link>
+      <!-- RIGHT WHEEL -->
 <joint name="right_wheel_joint" type="continuous">
     <parent link="base_link"/>
@@ -60,3 +61,17 @@
     </visual>
 </link>
+<joint name="castor_wheel_joint" type="continuous">
+    <parent link="chassis"/>
+    <child link="castor_wheel"/>
+    <origin xyz="0.24 0 0" />
+    <axis xyz="0 0 1"/>
+</joint>
+<link name="left_wheel">
+    <visual>
+        <geometry>
+            <sphere radius="0.05" />
+        </geometry>
+        <material name="black"/>
+    </visual>
+</link>
 </robot>

Commit message: adding collisions

File: description/robot_core.xacro (robot description, xacro)
@@ -30,4 +30,10 @@
             <material name="white"/>
         </visual>
+        <collision>
+            xacro <origin xyz="0.15 0 0.075"/>
+            xacro <geometry>
+                xacro <box size ="0.3 0.3 0.15"/>
+            </geometry>
+        </collision>
     </link>
       <!-- LEFT WHEEL -->
@@ -45,4 +51,9 @@
         <material name="blue"/>
     </visual>
+    <collision>
+        <geometry>
+            <cylinder length="0.04" radius="0.05" />
+        </geometry>
+    </collision>
 </link>
       <!-- RIGHT WHEEL -->
@@ -60,5 +71,11 @@
         <material name="blue"/>
     </visual>
+    <collision>
+        <geometry>
+            <cylinder length="0.04" radius="0.05" />
+        </geometry>
+    </collision>
 </link>
+ <!-- CASTOR WHEEL -->
 <joint name="castor_wheel_joint" type="continuous">
     <parent link="chassis"/>
@@ -67,5 +84,5 @@
     <axis xyz="0 0 1"/>
 </joint>
-<link name="left_wheel">
+<link name="castor_wheel">
     <visual>
         <geometry>
@@ -74,4 +91,9 @@
         <material name="black"/>
     </visual>
+    <collision>
+        <geometry>
+            <sphere radius="0.05" />
+        </geometry>
+    </collision>
 </link>
 </robot>

Commit message: uodates

File: description/robot_core.xacro (robot description, xacro)
@@ -1,4 +1,5 @@
 <?xml version="1.0"?>
 <robot xmlns:xacro="http://www.ros.org/wiki/xacro" >
+    xacro:<xacro:include filename="inertial_macros.xacro"/>
     xacro <material name="white">
         xacro <color rgba="1.0 1.0 1.0 1.0"/>
@@ -36,4 +37,7 @@
             </geometry>
         </collision>
+        <xacro:inertial_box mass="0.5" x="0.3" y="0.3" z="0.15">
+            <origin xyz="0.15 0 0.075"/>
+        </xacro:inertial_box>
     </link>
       <!-- LEFT WHEEL -->
@@ -56,4 +60,7 @@
         </geometry>
     </collision>
+    <xacro:inertial_cylinder mass ="0.1" length="0.04" radius="0.05">
+        <origin xyz="0 0 0" rpy="0 0 0" />
+    </xacro:inertial_cylinder>
 </link>
       <!-- RIGHT WHEEL -->
@@ -76,4 +83,7 @@
         </geometry>
     </collision>
+    <xacro:inertial_cylinder mass ="0.1" length="0.04" radius="0.05">
+        <origin xyz="0 0 0" rpy="0 0 0" />
+    </xacro:inertial_cylinder>
 </link>
  <!-- CASTOR WHEEL -->
@@ -96,4 +106,7 @@
         </geometry>
     </collision>
+    <xacro:inertial_sphere mass="0.1" radius="0.05">
+        <origin xyz = "0 0 0" rpy="0 0 0"/>
+    </xacro:inertial_sphere>
 </link>
 </robot>

Commit message: mods

File: description/robot_core.xacro (robot description, xacro)
@@ -41,4 +41,7 @@
         </xacro:inertial_box>
     </link>
+    <gazebo reference="chassis">
+        <material>Gazebo/white</material>
+    </gazebo>
       <!-- LEFT WHEEL -->
 <joint name="left_wheel_joint" type="continuous">
@@ -64,4 +67,7 @@
     </xacro:inertial_cylinder>
 </link>
+<gazebo reference="left_wheel">
+    <material>Gazebo/blue</material>
+</gazebo>
       <!-- RIGHT WHEEL -->
 <joint name="right_wheel_joint" type="continuous">
@@ -87,4 +93,7 @@
     </xacro:inertial_cylinder>
 </link>
+<gazebo reference="right_wheel">
+    <material>Gazebo/blue</material>
+</gazebo>
  <!-- CASTOR WHEEL -->
 <joint name="castor_wheel_joint" type="continuous">
@@ -110,3 +119,6 @@
     </xacro:inertial_sphere>
 </link>
+<gazebo reference="castor_wheel">
+    <material>Gazebo/black</material>
+</gazebo>
 </robot>

Commit message: adding colours for gazebo

File: description/robot_core.xacro (robot description, xacro)
@@ -42,5 +42,5 @@
     </link>
     <gazebo reference="chassis">
-        <material>Gazebo/white</material>
+        <material>Gazebo/White</material>
     </gazebo>
       <!-- LEFT WHEEL -->
@@ -68,5 +68,5 @@
 </link>
 <gazebo reference="left_wheel">
-    <material>Gazebo/blue</material>
+    <material>Gazebo/Blue</material>
 </gazebo>
       <!-- RIGHT WHEEL -->
@@ -94,5 +94,5 @@
 </link>
 <gazebo reference="right_wheel">
-    <material>Gazebo/blue</material>
+    <material>Gazebo/Blue</material>
 </gazebo>
  <!-- CASTOR WHEEL -->
@@ -120,5 +120,5 @@
 </link>
 <gazebo reference="castor_wheel">
-    <material>Gazebo/black</material>
+    <material>Gazebo/Black</material>
 </gazebo>
 </robot>
