Commit message: reverting to older

File: description/robot.urdf.xacro (robot description, xacro)
@@ -1,4 +1,4 @@
 <?xml version="1.0"?>
 <robot xmlns:xacro="http://www.ros.org/wiki/xacro"  name="robot">
-   <xacro:inlcude filename="robot_core.xacro" />
+  <link name="base_link"></link>
 </robot>

Commit message: Trying xacro again

File: description/robot.urdf.xacro (robot description, xacro)
@@ -1,4 +1,4 @@
 <?xml version="1.0"?>
 <robot xmlns:xacro="http://www.ros.org/wiki/xacro"  name="robot">
-  <link name="base_link"></link>
+  xacro:<xacro:include filename="robot_core.xacro"/>
 </robot>

Commit message: adding lidar files

File: description/robot.urdf.xacro (robot description, xacro)
@@ -3,3 +3,4 @@
   xacro:<xacro:include filename="robot_core.xacro"/>
   xacro:<xacro:include filename="gazebo_control.xacro"/>
+  xacro:<xacro:include filename="lidar.xacro"/>
 </robot>

File: description/robot_core.xacro (robot description, xacro)
@@ -13,4 +13,7 @@
     xacro <material name="black">
         xacro <color rgba="0 0 0 1"/>
+    </material>
+    xacro <material name="red">
+        xacro <color rgba="1 0 0 1"/>
     </material>
     <!-- BASE LINK -->
